Commit message: fix height of lider

File: simple_move.dummy_odom.urdf (robot description, URDF)
Before this commit: robot Simple, 3 links, 2 joints
Joints:
- joint fixed_main_to_baselaser_link: origin xyz=0.2 0.0 0.05 rpy=0 0 0 -> xyz=0.2 0.0 0.15 rpy=0 0 0

File: simple_move.urdf (robot description, URDF)
Before this commit: robot Simple, 3 links, 2 joints
Joints:
- joint fixed_main_to_baselaser_link: origin xyz=0.2 0.0 0.05 rpy=0 0 0 -> xyz=0.2 0.0 0.15 rpy=0 0 0
