Commit message: fix package-name

File: model/arm.urdf (robot description, URDF)
Before this commit: robot BodyBuilder, 10 links, 9 joints
Links:
- link GRIPPER0_lk: geometry collision cylinder length=0.040000000000000001 radius=0.016; collision mesh filename=package://irsl_mobile_arm/model/BodyBuilder_GRIPPER0_lk.stl
- link GRIPPER1_lk: geometry collision cylinder length=0.040000000000000001 radius=0.016; collision mesh filename=package://irsl_mobile_arm/model/BodyBuilder_GRIPPER1_lk.stl

File: model/base_arm.urdf (robot description, URDF)
Before this commit: robot base_arm, 14 links, 13 joints
Links:
- link GRIPPER0_lk: geometry collision cylinder length=0.040000000000000001 radius=0.016; collision mesh filename=package://irsl_mobile_arm/model/BodyBuilder_GRIPPER0_lk.stl
- link GRIPPER1_lk: geometry collision cylinder length=0.040000000000000001 radius=0.016; collision mesh filename=package://irsl_mobile_arm/model/BodyBuilder_GRIPPER1_lk.stl
