Commit message: update urdf model

File: model/base_arm.urdf (robot description, URDF)
Before this commit: robot base_arm, 14 links, 13 joints
Links:
- added link arm_camera_frame
- added link arm_camera_link
- added link base_camera_frame
- added link base_camera_link
- added link hand_camera_frame
- added link hand_camera_link
Joints:
- added joint arm_camera_frame_fixed_joint: type fixed, parent arm_camera_link, child arm_camera_frame, origin xyz=0 0 0 rpy=-1.5707963267948966 0 -1.5707963267948966
- added joint base_camera_frame_fixed_joint: type fixed, parent base_camera_link, child base_camera_frame, origin xyz=0 0 0 rpy=-1.5707963267948966 0 -1.5707963267948966
- added joint fixed_main_to_arm_camera_link: type fixed, parent ELBOW_Y_lk, child arm_camera_link, origin xyz=-0.1 0.12 0 rpy=-1.5707963267948966 0 1.5707963267948966
- added joint fixed_main_to_base_camera_link: type fixed, parent main, child base_camera_link, origin xyz=0.2 0.0 0.15 rpy=0 0 0
- added joint fixed_main_to_hand_camera_link: type fixed, parent WRIST_Y_lk, child hand_camera_link, origin xyz=-0.07 0.025 0 rpy=-1.5707963267948966 0 1.5707963267948966
- added joint hand_camera_frame_fixed_joint: type fixed, parent hand_camera_link, child hand_camera_frame, origin xyz=0 0 0 rpy=-1.5707963267948966 0 -1.5707963267948966

File: model/base_arm.urdf.xacro (robot description, xacro)
@@ -18,3 +18,28 @@
     </plugin>
   </gazebo>
+  <xacro:include filename="gazebo_plugins.xacro" />
+  <link name="base_camera_link" />
+  <joint name="fixed_main_to_base_camera_link" type="fixed">
+    <parent link="main"/>
+    <child link="base_camera_link"/>
+    <origin rpy="0 0 0" xyz="0.2 0.0 0.15"/>
+  </joint>
+  <link name="arm_camera_link" />
+  <joint name="fixed_main_to_arm_camera_link" type="fixed">
+    <parent link="ELBOW_Y_lk"/>
+    <child  link="arm_camera_link"/>
+    <origin xyz="-0.1 0.12 0" rpy="-1.5707963267948966 0 1.5707963267948966"/>
+  </joint>
+  <link name="hand_camera_link" />
+  <joint name="fixed_main_to_hand_camera_link" type="fixed">
+    <parent link="WRIST_Y_lk"/>
+    <child  link="hand_camera_link"/>
+    <origin xyz="-0.07 0.025 0" rpy="-1.5707963267948966 0 1.5707963267948966"/>
+  </joint>
+  <xacro:add_gazebo_camera camera_name="base_camera" frame="base_camera_frame" link_name="base_camera_link"
+                           rpy="-1.5707963267948966 0 -1.5707963267948966"/>
+  <xacro:add_gazebo_camera camera_name="arm_camera"  frame="arm_camera_frame"  link_name="arm_camera_link"
+                           rpy="-1.5707963267948966 0 -1.5707963267948966"/>
+  <xacro:add_gazebo_camera camera_name="hand_camera" frame="hand_camera_frame" link_name="hand_camera_link"
+                           rpy="-1.5707963267948966 0 -1.5707963267948966"/>
 </robot>

File: model/simple_move.urdf (robot description, URDF)
Before this commit: robot Simple, 3 links, 2 joints
Links:
- link main: mass 2.5 -> 10.0

Commit message: update urdf

File: model/base_arm.urdf (robot description, URDF)
Before this commit: robot base_arm, 20 links, 19 joints
Links:
- link main: mass 2.5 -> 40.0

File: model/simple_move.urdf (robot description, URDF)
Before this commit: robot Simple, 3 links, 2 joints
Links:
- link main: mass 10.0 -> 40.0
